File: v2/keeb2.kicad_pcb (KiCad board)
At the start: 2 copper layers, 306.7 x 100.9 mm, 160 parts, among them J1 AVR-ISP-6, J3 AudioJack4, SW10 SW_Push, SW11 SW_Push, SW12 SW_Push, SW13 SW_Push, SW14 SW_Push, SW15 SW_Push, SW16 SW_Push, SW17 SW_Push, SW18 SW_Push, SW19 SW_Push, SW2 SW_Push_Reset, SW20 SW_Push, SW21 SW_Push, SW22 SW_Push, SW23 SW_Push, SW24 SW_Push, SW25 SW_Push, SW26 SW_Push, SW27 SW_Push, SW28 SW_Push, SW29 SW_Push, SW3 SW_Push, SW30 SW_Push, SW31 SW_Push, SW32 SW_Push, SW33 SW_Push, SW34 SW_Push, SW35 SW_Push, SW36 SW_Push, SW37 SW_Push, SW38 SW_Push, SW39 SW_Push, SW4 SW_Push, SW40 SW_Push, SW41 SW_Push, SW42 SW_Push, SW43 SW_Push, SW44 SW_Push, SW45 SW_Push, SW46 SW_Push, SW47 SW_Push, SW48 SW_Push, SW49 SW_Push, SW5 SW_Push, SW50 SW_Push, SW51 SW_Push, SW52 SW_Push, SW53 SW_Push, SW54 SW_Push, SW55 SW_Push, SW56 SW_Push, SW57 SW_Push, SW58 SW_Push, SW59 SW_Push, SW6 SW_Push, SW60 SW_Push, SW61 SW_Push, SW62 SW_Push, SW63 SW_Push, SW64 SW_Push, SW65 SW_Push, SW66 SW_Push, SW67 SW_Push, SW68 SW_Push, SW69 SW_Push, SW7 SW_Push, SW70 SW_Push, SW71 RotaryEncoder_Switch, SW8 SW_Push, SW9 SW_Push, U1 ATmega32U4-A, Y1 XTAL

Commit message: Changed switch value for better understanding in PCB view
Parts:
- SW10: value SW_Push -> KC_7
- SW11: value SW_Push -> KC_8
- SW12: value SW_Push -> KC_9
- SW13: value SW_Push -> KC_0
- SW14: value SW_Push -> KC_MINUS
- SW15: value SW_Push -> KC_EQUAL
- SW16: value SW_Push -> KC_BACKSPACE
- SW17: value SW_Push -> KC_TAB
- SW18: value SW_Push -> KC_Q
- SW19: value SW_Push -> KC_W
- SW20: value SW_Push -> KC_E
- SW21: value SW_Push -> KC_R
- SW22: value SW_Push -> KC_T
- SW23: value SW_Push -> KC_Y
- SW24: value SW_Push -> KC_U
- SW25: value SW_Push -> KC_I
- SW26: value SW_Push -> KC_O
- SW27: value SW_Push -> KC_P
- SW28: value SW_Push -> KC_LEFT_BRACKET
- SW29: value SW_Push -> KC_RIGHT_BRACKET
- SW3: value SW_Push -> KC_ESCAPE
- SW30: value SW_Push -> KC_DEL
- SW31: value SW_Push -> KC_CAPS
- SW32: value SW_Push -> KC_A
- SW33: value SW_Push -> KC_S
- SW34: value SW_Push -> KC_D
- SW35: value SW_Push -> KC_F
- SW36: value SW_Push -> KC_G
- SW37: value SW_Push -> KC_H
- SW38: value SW_Push -> KC_J
- SW39: value SW_Push -> KC_K
- SW4: value SW_Push -> KC_1
- SW40: value SW_Push -> KC_L
- SW41: value SW_Push -> KC_SEMICOLON
- SW42: value SW_Push -> KC_QUOTE
- SW43: value SW_Push -> KC_NONUS_HASH
- SW44: value SW_Push -> KC_ENTER
- SW45: value SW_Push -> KC_PAGE_UP
- SW46: value SW_Push -> KC_LEFT_SHIFT
- SW47: value SW_Push -> KC_GRAVE
- SW48: value SW_Push -> KC_Z
- SW49: value SW_Push -> KC_X
- SW5: value SW_Push -> KC_2
- SW50: value SW_Push -> KC_C
- SW51: value SW_Push -> KC_V
- SW52: value SW_Push -> KC_B
- SW53: value SW_Push -> KC_N
- SW54: value SW_Push -> KC_M
- SW55: value SW_Push -> KC_COMMA
- SW56: value SW_Push -> KC_DOT
- SW57: value SW_Push -> KC_SLASH
- SW58: value SW_Push -> KC_RIGHT_SHIFT
- SW59: value SW_Push -> KC_UP
- SW6: value SW_Push -> KC_3
- SW60: value SW_Push -> KC_PAGE_DOWN
- SW61: value SW_Push -> KC_LEFT_CTRL
- SW62: value SW_Push -> KC_LEFT_GUI
- SW63: value SW_Push -> KC_LEFT_ALT
- SW64: value SW_Push -> KC_SPACE
- SW65: value SW_Push -> KC_RIGHT_ALT
- SW66: value SW_Push -> KC_RIGHT_GUI
- SW67: value SW_Push -> KC_RIGHT_CTRL
- SW68: value SW_Push -> KC_LEFT
- SW69: value SW_Push -> KC_DOWN
- SW7: value SW_Push -> KC_4
- SW70: value SW_Push -> KC_RIGHT
- SW8: value SW_Push -> KC_5
- SW9: value SW_Push -> KC_6
Changed lines of the file:
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@@
 			)
 		)
-		(property "Value" "SW_Push"
+		(property "Value" "KC_COMMA"
 			(at 0 -7.9375 0)
 			(layer "Dwgs.User")
@@
 			)
 		)
-		(property "Value" "SW_Push"
+		(property "Value" "KC_0"
 			(at 0 -7.9375 0)
 			(layer "Dwgs.User")
@@
 			)
 		)
-		(property "Value" "SW_Push"
+		(property "Value" "KC_E"
 			(at 0 -7.9375 0)
 			(layer "Dwgs.User")
@@
 			)
 		)
-		(property "Value" "SW_Push"
+		(property "Value" "KC_Q"
 			(at 0 -7.9375 0)
 			(layer "Dwgs.User")
@@
 			)
 		)
-		(property "Value" "SW_Push"
+		(property "Value" "KC_LEFT_SHIFT"
 			(at 0 -7.9375 0)
 			(layer "Dwgs.User")
@@
 			)
 		)
-		(property "Value" "SW_Push"
+		(property "Value" "KC_RIGHT"
 			(at 0 -7.9375 0)
 			(layer "Dwgs.User")
@@
 			)
 		)
-		(property "Value" "SW_Push"
+		(property "Value" "KC_7"
 			(at 0 -7.9375 0)
 			(layer "Dwgs.User")
@@
 			)
 		)
-		(property "Value" "SW_Push"
+		(property "Value" "KC_SEMICOLON"
 			(at 0 -7.9375 0)
 			(layer "Dwgs.User")
@@
 			)
 		)
-		(property "Value" "SW_Push"
+		(property "Value" "KC_EQUAL"
 			(at 0 -7.9375 0)
 			(layer "Dwgs.User")
@@
 			)
 		)
-		(property "Value" "SW_Push"
+		(property "Value" "KC_8"
 			(at 0 -7.9375 0)
 			(layer "Dwgs.User")
@@
 			)
 		)
-		(property "Value" "SW_Push"
+		(property "Value" "KC_RIGHT_CTRL"
 			(at 0 -7.9375 0)
 			(layer "Dwgs.User")
@@
 			)
 		)
-		(property "Value" "SW_Push"
+		(property "Value" "KC_LEFT"
 			(at 0 -7.9375 0)
 			(layer "Dwgs.User")
@@
 			)
 		)
-		(property "Value" "SW_Push"
+		(property "Value" "KC_U"
 			(at 0 -7.9375 0)
 			(layer "Dwgs.User")
@@
 			)
 		)
-		(property "Value" "SW_Push"
+		(property "Value" "KC_M"
 			(at 0 -7.9375 0)
 			(layer "Dwgs.User")
@@
 			)
 		)
-		(property "Value" "SW_Push"
+		(property "Value" "KC_MINUS"
 			(at 0 -7.9375 0)
 			(layer "Dwgs.User")
@@
 			)
 		)
-		(property "Value" "SW_Push"
+		(property "Value" "KC_RIGHT_BRACKET"
 			(at 0 -7.9375 0)
 			(layer "Dwgs.User")
@@
 			)
 		)
-		(property "Value" "SW_Push"
+		(property "Value" "KC_BACKSPACE"
 			(at 0 -7.9375 0)
 			(layer "Dwgs.User")
@@
 			)
 		)
-		(property "Value" "SW_Push"
+		(property "Value" "KC_ESCAPE"
 			(at 0 -7.9375 0)
 			(layer "Dwgs.User")
@@
 			)
 		)
-		(property "Value" "SW_Push"
+		(property "Value" "KC_W"
 			(at 0 -7.9375 0)
 			(layer "Dwgs.User")
@@
 			)
 		)
-		(property "Value" "SW_Push"
+		(property "Value" "KC_LEFT_GUI"
 			(at 0 -7.9375 0)
 			(layer "Dwgs.User")
@@
 			)
 		)
-		(property "Value" "SW_Push"
+		(property "Value" "KC_UP"
 			(at 0 -7.9375 0)
 			(layer "Dwgs.User")
@@
 			)
 		)
-		(property "Value" "SW_Push"
+		(property "Value" "KC_LEFT_CTRL"
 			(at 0 -7.9375 0)
 			(layer "Dwgs.User")
@@
 			)
 		)
-		(property "Value" "SW_Push"
+		(property "Value" "KC_QUOTE"
 			(at 0 -7.9375 0)
 			(layer "Dwgs.User")
@@
 			)
 		)
-		(property "Value" "SW_Push"
+		(property "Value" "KC_H"
 			(at 0 -7.9375 0)
 			(layer "Dwgs.User")
@@
 			)
 		)
-		(property "Value" "SW_Push"
+		(property "Value" "KC_NONUS_HASH"
 			(at 0 -7.9375 0)
 			(layer "Dwgs.User")
@@
 			)
 		)
-		(property "Value" "SW_Push"
+		(property "Value" "KC_B"
 			(at 0 -7.9375 0)
 			(layer "Dwgs.User")
@@
 			)
 		)
-		(property "Value" "SW_Push"
+		(property "Value" "KC_DOWN"
 			(at 0 -7.9375 0)
 			(layer "Dwgs.User")
@@
 			)
 		)
-		(property "Value" "SW_Push"
+		(property "Value" "KC_CAPS"
 			(at 0 -7.9375 0)
 			(layer "Dwgs.User")
@@
 			)
 		)
-		(property "Value" "SW_Push"
+		(property "Value" "KC_3"
 			(at 0 -7.9375 0)
 			(layer "Dwgs.User")
@@
 			)
 		)
-		(property "Value" "SW_Push"
+		(property "Value" "KC_2"
 			(at 0 -7.9375 0)
 			(layer "Dwgs.User")
@@
 			)
 		)
-		(property "Value" "SW_Push"
+		(property "Value" "KC_RIGHT_ALT"
 			(at 0 -7.9375 0)
 			(layer "Dwgs.User")
@@
 			)
 		)
-		(property "Value" "SW_Push"
+		(property "Value" "KC_TAB"
 			(at 0 -7.9375 0)
 			(layer "Dwgs.User")
@@
 			)
 		)
-		(property "Value" "SW_Push"
+		(property "Value" "KC_RIGHT_GUI"
 			(at 0 -7.9375 0)
 			(layer "Dwgs.User")
@@
 			)
 		)
-		(property "Value" "SW_Push"
+		(property "Value" "KC_N"
 			(at 0 -7.9375 0)
 			(layer "Dwgs.User")
@@
 			)
 		)
-		(property "Value" "SW_Push"
+		(property "Value" "KC_DOT"
 			(at 0 -7.9375 0)
 			(layer "Dwgs.User")
@@
 			)
 		)
-		(property "Value" "SW_Push"
+		(property "Value" "KC_A"
 			(at 0 -7.9375 0)
 			(layer "Dwgs.User")
@@
 			)
 		)
-		(property "Value" "SW_Push"
+		(property "Value" "KC_RIGHT_SHIFT"
 			(at 0 -7.9375 0)
 			(layer "Dwgs.User")
@@
 			)
 		)
-		(property "Value" "SW_Push"
+		(property "Value" "KC_P"
 			(at 0 -7.9375 0)
 			(layer "Dwgs.User")
@@
 			)
 		)
-		(property "Value" "SW_Push"
+		(property "Value" "KC_GRAVE"
 			(at 0 -7.9375 0)
 			(layer "Dwgs.User")
@@
 			)
 		)
-		(property "Value" "SW_Push"
+		(property "Value" "KC_ENTER"
 			(at 0 -7.9375 0)
 			(layer "Dwgs.User")
@@
 			)
 		)
-		(property "Value" "SW_Push"
+		(property "Value" "KC_X"
 			(at 0 -7.9375 0)
 			(layer "Dwgs.User")
@@
 			)
 		)
-		(property "Value" "SW_Push"
+		(property "Value" "KC_R"
 			(at 0 -7.9375 0)
 			(layer "Dwgs.User")
@@
 			)
 		)
-		(property "Value" "SW_Push"
+		(property "Value" "KC_L"
 			(at 0 -7.9375 0)
 			(layer "Dwgs.User")
@@
 			)
 		)
-		(property "Value" "SW_Push"
+		(property "Value" "KC_5"
 			(at 0 -7.9375 0)
 			(layer "Dwgs.User")
@@
 			)
 		)
-		(property "Value" "SW_Push"
+		(property "Value" "KC_6"
 			(at 0 -7.9375 0)
 			(layer "Dwgs.User")
@@
 			)
 		)
-		(property "Value" "SW_Push"
+		(property "Value" "KC_DEL"
 			(at 0 -7.9375 0)
 			(layer "Dwgs.User")
@@
 			)
 		)
-		(property "Value" "SW_Push"
+		(property "Value" "KC_SPACE"
 			(at 0 -7.9375 0)
 			(layer "Dwgs.User")
@@
 			)
 		)
-		(property "Value" "SW_Push"
+		(property "Value" "KC_SLASH"
 			(at 0 -7.9375 0)
 			(layer "Dwgs.User")
@@
 			)
 		)
-		(property "Value" "SW_Push"
+		(property "Value" "KC_F"
 			(at 0 -7.9375 0)
 			(layer "Dwgs.User")
@@
 			)
 		)
-		(property "Value" "SW_Push"
+		(property "Value" "KC_PAGE_UP"
 			(at 0 -7.9375 0)
 			(layer "Dwgs.User")
@@
 			)
 		)
-		(property "Value" "SW_Push"
+		(property "Value" "KC_K"
 			(at 0 -7.9375 0)
 			(layer "Dwgs.User")
@@
 			)
 		)
-		(property "Value" "SW_Push"
+		(property "Value" "KC_J"
 			(at 0 -7.9375 0)
 			(layer "Dwgs.User")
@@
 			)
 		)
-		(property "Value" "SW_Push"
+		(property "Value" "KC_LEFT_BRACKET"
 			(at 0 -7.9375 0)
 			(layer "Dwgs.User")
@@
 			)
 		)
-		(property "Value" "SW_Push"
+		(property "Value" "KC_4"
 			(at 0 -7.9375 0)
 			(layer "Dwgs.User")
@@
 			)
 		)
-		(property "Value" "SW_Push"
+		(property "Value" "KC_C"
 			(at 0 -7.9375 0)
 			(layer "Dwgs.User")
@@
 			)
 		)
-		(property "Value" "SW_Push"
+		(property "Value" "KC_I"
 			(at 0 -7.9375 0)
 			(layer "Dwgs.User")
@@
 			)
 		)
-		(property "Value" "SW_Push"
+		(property "Value" "KC_V"
 			(at 0 -7.9375 0)
 			(layer "Dwgs.User")
@@
 			)
 		)
-		(property "Value" "SW_Push"
+		(property "Value" "KC_Z"
 			(at 0 -7.9375 0)
 			(layer "Dwgs.User")
@@
 			)
 		)
-		(property "Value" "SW_Push"
+		(property "Value" "KC_D"
 			(at 0 -7.9375 0)
 			(layer "Dwgs.User")
@@
 			)
 		)
-		(property "Value" "SW_Push"
+		(property "Value" "KC_O"
 			(at 0 -7.9375 0)
 			(layer "Dwgs.User")
@@
 			)
 		)
-		(property "Value" "SW_Push"
+		(property "Value" "KC_T"
 			(at 0 -7.9375 0)
 			(layer "Dwgs.User")
@@
 			)
 		)
-		(property "Value" "SW_Push"
+		(property "Value" "KC_Y"
 			(at 0 -7.9375 0)
 			(layer "Dwgs.User")
@@
 			)
 		)
-		(property "Value" "SW_Push"
+		(property "Value" "KC_9"
 			(at 0 -7.9375 0)
 			(layer "Dwgs.User")
@@
 			)
 		)
-		(property "Value" "SW_Push"
+		(property "Value" "KC_1"
 			(at 0 -7.9375 0)
 			(layer "Dwgs.User")
@@
 			)
 		)
-		(property "Value" "SW_Push"
+		(property "Value" "KC_PAGE_DOWN"
 			(at 0 -7.9375 0)
 			(layer "Dwgs.User")
@@
 			)
 		)
-		(property "Value" "SW_Push"
+		(property "Value" "KC_LEFT_ALT"
 			(at 0 -7.9375 0)
 			(layer "Dwgs.User")
@@
 			)
 		)
-		(property "Value" "SW_Push"
+		(property "Value" "KC_G"
 			(at 0 -7.9375 0)
 			(layer "Dwgs.User")
@@
 			)
 		)
-		(property "Value" "SW_Push"
+		(property "Value" "KC_S"
 			(at 0 -7.9375 0)
 			(layer "Dwgs.User")

Commit message: Changed switch footprint to MX footprint
Realised I didn't want Alp switch so changed to more classic MX switch.
Need a full redone of the routing :'(
Parts:
- SW10, SW11, SW12, SW13, SW14, SW15, SW18, SW19, SW20, SW21, SW22, SW23, SW24, SW25, SW26, SW27, SW28, SW29, SW3, SW30, SW32, SW33, SW34, SW35, SW36, SW37, SW38, SW39, SW4, SW40, SW41, SW42, SW43, SW45, SW47, SW48, SW49, SW5, SW50, SW51, SW52, SW53, SW54, SW55, SW56, SW57, SW59, SW6, SW60, SW65, SW66, SW67, SW68, SW69, SW7, SW70, SW8, SW9: footprint Alps_Only:ALPS-1U -> Button_Switch_Keyboard:SW_Cherry_MX_1.00u_PCB
- SW16: footprint Alps_Only:ALPS-2U -> Button_Switch_Keyboard:SW_Cherry_MX_2.00u_PCB
- SW17: footprint Alps_Only:ALPS-1.5U -> Button_Switch_Keyboard:SW_Cherry_MX_1.50u_PCB
- SW31, SW58: footprint Alps_Only:ALPS-1.75U -> Button_Switch_Keyboard:SW_Cherry_MX_1.75u_PCB
- SW44: footprint Alps_Only:ALPS-ISO -> Button_Switch_Keyboard:SW_Cherry_MX_ISOEnter_PCB
- SW46, SW61, SW62, SW63: footprint Alps_Only:ALPS-1.25U -> Button_Switch_Keyboard:SW_Cherry_MX_1.25u_PCB
- SW64: footprint Alps_Only:ALPS-6.25U -> Button_Switch_Keyboard:SW_Cherry_MX_6.25u_PCB
- moved C1 87.2 mm to (208.3, 248.2)
- moved C3 87.2 mm to (227.4, 260.8)
- moved C4 87.2 mm to (200.6, 263.7)
- moved J1 87.2 mm to (238.4, 262.8)
- moved R1 87.2 mm to (203.2, 267.1)
- moved R2 87.2 mm to (219.2, 250.6)
- moved Y1 87.2 mm to (222.8, 259.6)
- moved C2 87.2 mm to (227.4, 258.0)
- moved C5 87.2 mm to (201.5, 251.6)
- moved C6 87.2 mm to (214.5, 267.1)
- moved C7 87.2 mm to (220.3, 254.7)
- moved SW2 87.2 mm to (238.6, 253.7)
- moved U1 87.2 mm to (208.7, 259.4)
- moved D2 21.5 mm to (88.6, 102.9)
- moved D42 10.3 mm to (319.2, 141.1)
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Routing:
- net GND: track 565.4 -> 214.9 mm, vias 11 -> 8
- net +5V: track 526.5 -> 211.0 mm, vias 8 -> 7
- net col14: track 234.4 -> 5.46 mm, vias 2 -> 0
- net col13: track 226.1 -> 6.91 mm, vias 1 -> 0
- net col12: track 211.5 -> 6.08 mm, vias 1 -> 0
- net col0: track 228.5 -> 24.0 mm
- net Rota_B: track 202.0 -> 13.0 mm, vias 2 -> 0
- net col1: track 211.4 -> 22.4 mm
- net col11: track 193.7 -> 10.5 mm, vias 1 -> 0
- net Rota_A: track 196.4 -> 14.7 mm, vias 2 -> 0
- net SDA: track 183.5 -> 11.0 mm
- net SCL: track 176.4 -> 9.18 mm
- net col2: track 186.2 -> 20.8 mm
- net SCK: track 182.3 -> 30.0 mm, vias 1 -> 0
- net col3: track 170.2 -> 19.1 mm
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Other:
- board size 306.7 x 100.9 mm -> 306.7 x 97.5 mm

Commit message: Linked part of the design; need to move reset button &  ISP
Parts:
- moved C1 84.8 mm to (216.7, 163.8)
- moved C3 84.8 mm to (235.8, 176.4)
- moved C4 84.8 mm to (209.0, 179.3)
- moved J1 84.8 mm to (246.9, 178.4)
- moved R1 84.8 mm to (211.6, 182.7)
- moved C5 84.8 mm to (209.9, 167.2)
- moved C6 84.8 mm to (223.0, 182.7)
- moved C7 84.8 mm to (228.7, 170.3)
- moved R2 84.8 mm to (227.7, 166.2)
- moved SW2 84.8 mm to (247.0, 169.3)
- moved Y1 84.8 mm to (231.2, 175.2)
- moved C2 84.8 mm to (235.8, 173.6)
- moved U1 84.8 mm to (217.1, 175.0)
Connections:
- U1 pad 39: row0 -> row2
- U1 pad 41: row2 -> row0
Routing:
- net +5V: track 211.0 -> 491.5 mm, vias 7 -> 8
- net GND: track 214.9 -> 492.0 mm
- net col0: track 24.0 -> 245.1 mm
- net col14: track 5.46 -> 210.6 mm, vias 0 -> 1
- net col1: track 22.4 -> 224.9 mm
- net col2: track 20.8 -> 201.8 mm
- net col3: track 19.1 -> 181.7 mm
- net D-: track 43.7 -> 196.7 mm
- net D+: track 44.2 -> 196.4 mm
- net col4: track 18.1 -> 161.9 mm
- net Rota_A: track 14.7 -> 148.6 mm
- net Rota_B: track 13.0 -> 145.7 mm
- net SCL: track 9.18 -> 141.7 mm
- net SDA: track 11.0 -> 142.7 mm
- net col5: track 15.0 -> 130.1 mm
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Other:
- board size 306.7 x 97.5 mm -> 307.7 x 103.5 mm

Commit message: Moved ISP and reset button. Finished routing
Moved the ISP IO to make it easier to route them to the MCU
Parts:
- J1: moved to F.Cu
- moved J1 80.8 mm to (166.1, 176.3), turned to 90 degrees
- moved SW2 69.2 mm to (178.2, 176.5), turned to 180 degrees
Connections:
- SW11 pad 2: MOSI -> col8
- SW12 pad 2: MISO -> col9
- SW13 pad 2: SCK -> col10
- SW19 pad 2: col2 -> MOSI
- SW20 pad 2: col3 -> MISO
- SW21 pad 2: col4 -> SCK
- SW25 pad 2: MOSI -> col8
- SW26 pad 2: MISO -> col9
- SW27 pad 2: SCK -> col10
- SW33 pad 2: col2 -> MOSI
- SW34 pad 2: col3 -> MISO
- SW35 pad 2: col4 -> SCK
- SW39 pad 2: MOSI -> col8
- SW40 pad 2: MISO -> col9
- SW41 pad 2: SCK -> col10
- SW48 pad 2: col2 -> MOSI
- SW49 pad 2: col3 -> MISO
- SW5 pad 2: col2 -> MOSI
- SW50 pad 2: col4 -> SCK
- SW54 pad 2: MOSI -> col8
- SW55 pad 2: MISO -> col9
- SW56 pad 2: SCK -> col10
- SW6 pad 2: col3 -> MISO
- SW63 pad 2: col2 -> MOSI
- SW65 pad 2: MISO -> col9
- SW66 pad 2: SCK -> col10
- SW7 pad 2: col4 -> SCK
- U1 pad 19: MOSI -> col8
- U1 pad 20: MISO -> col9
- U1 pad 21: SCK -> col10
- U1 pad 30: col2 -> MOSI
- U1 pad 31: col3 -> MISO
- U1 pad 32: col4 -> SCK
Routing:
- net col2: track 201.8 -> 0.00 mm, vias 1 -> 0
- net col3: track 181.7 -> 0.00 mm, vias 1 -> 0
- net col10: track 0.00 -> 164.0 mm, vias 0 -> 1
- net col4: track 161.9 -> 0.00 mm, vias 1 -> 0
- net col9: track 0.00 -> 147.6 mm
- net col13: track 87.1 -> 215.6 mm, vias 0 -> 1
- net col8: track 0.00 -> 125.9 mm, vias 0 -> 1
- net MOSI: track 94.9 -> 212.8 mm
- net col12: track 92.1 -> 201.4 mm, vias 0 -> 1
- net GND: track 492.0 -> 597.3 mm, vias 8 -> 13
- net col11: track 102.5 -> 183.5 mm, vias 0 -> 1
- net MISO: track 114.9 -> 185.6 mm, vias 0 -> 2
- net SCK: track 108.5 -> 164.6 mm, vias 0 -> 1
- net Rota_B: track 145.7 -> 200.7 mm, vias 0 -> 2
- net RESET: track 42.1 -> 96.9 mm, vias 0 -> 4
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- added copper zone on F.Cu, net GND
