File: v2/keeb2.kicad_pcb (KiCad board)
At the start: 2 copper layers, 307.7 x 103.5 mm, 160 parts, among them J1 AVR-ISP-6, J3 AudioJack4, SW10 KC_7, SW11 KC_8, SW12 KC_9, SW13 KC_0, SW14 KC_MINUS, SW15 KC_EQUAL, SW16 KC_BACKSPACE, SW17 KC_TAB, SW18 KC_Q, SW19 KC_W, SW2 SW_Push_Reset, SW20 KC_E, SW21 KC_R, SW22 KC_T, SW23 KC_Y, SW24 KC_U, SW25 KC_I, SW26 KC_O, SW27 KC_P, SW28 KC_LEFT_BRACKET, SW29 KC_RIGHT_BRACKET, SW3 KC_ESCAPE, SW30 KC_DEL, SW31 KC_CAPS, SW32 KC_A, SW33 KC_S, SW34 KC_D, SW35 KC_F, SW36 KC_G, SW37 KC_H, SW38 KC_J, SW39 KC_K, SW4 KC_1, SW40 KC_L, SW41 KC_SEMICOLON, SW42 KC_QUOTE, SW43 KC_NONUS_HASH, SW44 KC_ENTER, SW45 KC_PAGE_UP, SW46 KC_LEFT_SHIFT, SW47 KC_GRAVE, SW48 KC_Z, SW49 KC_X, SW5 KC_2, SW50 KC_C, SW51 KC_V, SW52 KC_B, SW53 KC_N, SW54 KC_M, SW55 KC_COMMA, SW56 KC_DOT, SW57 KC_SLASH, SW58 KC_RIGHT_SHIFT, SW59 KC_UP, SW6 KC_3, SW60 KC_PAGE_DOWN, SW61 KC_LEFT_CTRL, SW62 KC_LEFT_GUI, SW63 KC_LEFT_ALT, SW64 KC_SPACE, SW65 KC_RIGHT_ALT, SW66 KC_RIGHT_GUI, SW67 KC_RIGHT_CTRL, SW68 KC_LEFT, SW69 KC_DOWN, SW7 KC_4, SW70 KC_RIGHT, SW71 RotaryEncoder_Switch, SW8 KC_5, SW9 KC_6, U1 ATmega32U4-A, Y1 XTAL

Commit message: Change outline to fit new case
Add mounting holes at correct location

case height : 96 mm
pcb height : 95.5mm

case length : 305 mm
pcb length : 304.5 mm
Parts:
- added H1: MountingHole, MountingHole:MountingHole_2.1mm, F.Cu at (30.2, 33.2)
- added H10: MountingHole, MountingHole:MountingHole_2.1mm, F.Cu at (279.8, 70.2)
- added H2: MountingHole, MountingHole:MountingHole_2.1mm, F.Cu at (43.2, 14.8)
- added H3: MountingHole, MountingHole:MountingHole_2.1mm, F.Cu at (29.8, 85.2)
- added H4: MountingHole, MountingHole:MountingHole_2.1mm, F.Cu at (66.8, 60.8)
- added H5: MountingHole, MountingHole:MountingHole_2.1mm, F.Cu at (132.8, 51.8)
- added H6: MountingHole, MountingHole:MountingHole_2.1mm, F.Cu at (167.8, 34.2)
- added H7: MountingHole, MountingHole:MountingHole_2.1mm, F.Cu at (193.2, 80.2)
- added H8: MountingHole, MountingHole:MountingHole_2.1mm, F.Cu at (242.2, 14.2)
- added H9: MountingHole, MountingHole:MountingHole_2.1mm, F.Cu at (271.2, 33.2)
- moved D25 438.6 mm to (694.7, 144.5)
- moved C1 438.6 mm to (654.8, 186.1)
- moved C2 438.6 mm to (673.9, 195.9)
- moved C3 438.6 mm to (673.9, 198.7)
- moved C4 438.6 mm to (647.1, 201.6)
- moved C5 438.6 mm to (648.0, 189.5)
- moved C6 438.6 mm to (661.0, 205.0)
- moved C7 438.6 mm to (666.8, 192.6)
- moved D1 438.6 mm to (519.2, 122.1)
- moved D10 438.6 mm to (666.7, 125.3)
- moved D11 438.6 mm to (685.7, 125.3)
- moved D13 438.6 mm to (723.6, 125.3)
- moved D16 438.6 mm to (518.3, 144.3)
- moved D17 438.6 mm to (542.5, 144.3)
- moved D18 438.6 mm to (561.6, 144.3)
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Other:
- board size 307.7 x 103.5 mm -> 306.3 x 101.5 mm

Commit message: squeeze keyboard in case
removed colomn 14 (4 keys), TTRS connection, and rotary encoder
Parts:
- removed D29, D44, D59, D69: D, Diode_SMD:D_SOD-123
- removed J3: AudioJack4, Keebio-Parts:TRRS-PJ-320A
- removed R7, R8: 10k, Resistor_SMD:R_0805_2012Metric_Pad1.20x1.40mm_HandSolder
- removed SW30: KC_DEL, Button_Switch_Keyboard:SW_Cherry_MX_1.00u_PCB
- removed SW45: KC_PAGE_UP, Button_Switch_Keyboard:SW_Cherry_MX_1.00u_PCB
- removed SW60: KC_PAGE_DOWN, Button_Switch_Keyboard:SW_Cherry_MX_1.00u_PCB
- removed SW70: KC_RIGHT, Button_Switch_Keyboard:SW_Cherry_MX_1.00u_PCB
- removed SW71: RotaryEncoder_Switch, Keebio-Parts:RotaryEncoder_EC11
- D10, D11, D12, D13, D14, D15, D16, D17, D18, D19, D20, D21, D22, D23, D24, D25, D26, D27, D28, D3, D30, D31, D32, D33, D34, D35, D36, D37, D38, D39, D4, D40, D41, D42, D43, D45, D46, D47, D48, D49, D5, D50, D51, D52, D53, D54, D55, D56, D57, D58, D6, D60, D61, D62, D63, D64, D65, D66, D67, D68, D7, D8, D9: moved to F.Cu
- moved D68 666.4 mm to (162.2, -46.5), turned to 0 degrees
- moved D58 663.0 mm to (156.4, -39.8), turned to 0 degrees
- moved D15 660.8 mm to (139.0, -66.6), turned to 0 degrees
- moved D43 651.0 mm to (150.6, -49.8), turned to 0 degrees
- moved D67 650.2 mm to (162.2, -49.8), turned to 0 degrees
- moved D42 644.1 mm to (150.6, -53.2), turned to 0 degrees
- moved D28 640.7 mm to (144.8, -59.9), turned to 0 degrees
- moved D57 639.3 mm to (156.4, -43.1), turned to 0 degrees
- moved D14 634.4 mm to (139.0, -69.9), turned to 0 degrees
- moved D66 633.8 mm to (162.2, -53.2), turned to 0 degrees
- moved D41 627.1 mm to (150.6, -56.5), turned to 0 degrees
- moved D27 623.9 mm to (144.8, -63.2), turned to 0 degrees
- moved D65 617.8 mm to (162.2, -56.5), turned to 0 degrees
- moved D56 616.6 mm to (156.4, -46.5), turned to 0 degrees
- moved D13 612.1 mm to (133.2, -36.4), turned to 0 degrees
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Connections:
- U1 pad 10: Rota_B -> unconnected-(U1-PB2-Pad10)
- U1 pad 11: SCL -> unconnected-(U1-PB3-Pad11)
- U1 pad 12: SDA -> unconnected-(U1-PB7-Pad12)
- U1 pad 27: col14 -> unconnected-(U1-PD7-Pad27)
- U1 pad 9: Rota_A -> unconnected-(U1-PB1-Pad9)
Routing:
- net +5V: track 521.8 -> 92.2 mm, vias 9 -> 6
- net GND: track 597.3 -> 169.5 mm, vias 13 -> 7
- net row0: track 327.3 -> 10.0 mm, vias 2 -> 0
- net row2: track 318.9 -> 12.9 mm, vias 6 -> 0
- net row4: track 305.3 -> 0.00 mm, vias 2 -> 0
- net row1: track 315.8 -> 11.3 mm, vias 2 -> 0
- net row3: track 297.7 -> 5.61 mm, vias 6 -> 1
- net col0: track 245.1 -> 5.99 mm, vias 1 -> 0
- net col1: track 224.9 -> 5.32 mm, vias 1 -> 0
- net col13: track 215.6 -> 4.80 mm, vias 1 -> 0
- net col14: track 210.6 -> 0.00 mm, vias 1 -> 0
- net MOSI: track 212.8 -> 4.66 mm, vias 2 -> 0
- net Rota_B: track 200.7 -> 0.00 mm, vias 2 -> 0
- net Rota_A: track 195.5 -> 0.00 mm, vias 2 -> 0
- net col12: track 201.4 -> 6.08 mm, vias 1 -> 0
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Other:
- board size 306.3 x 101.5 mm -> 304.5 x 101.5 mm

Commit message: Finished routing
Parts:
- D10, D11, D12, D13, D14, D15, D16, D17, D18, D19, D20, D21, D22, D23, D24, D25, D26, D27, D28, D3, D30, D31, D32, D33, D34, D35, D36, D37, D38, D39, D4, D40, D41, D42, D43, D45, D46, D47, D48, D49, D5, D50, D51, D52, D53, D54, D55, D56, D57, D58, D6, D60, D61, D62, D63, D64, D65, D66, D67, D68, D7, D8, D9: moved to B.Cu
- moved D61 191.8 mm to (49.7, 85.4), turned to 90 degrees
- moved D68 180.2 mm to (295.8, 74.5)
- moved D60 179.0 mm to (25.2, 85.3), turned to 90 degrees
- moved D67 178.1 mm to (285.6, 78.7), turned to -90 degrees
- moved D62 175.7 mm to (73.9, 85.3), turned to 90 degrees
- moved D45 169.3 mm to (21.3, 62.8), turned to -90 degrees
- moved D66 168.1 mm to (266.5, 78.7), turned to -90 degrees
- moved D58 167.0 mm to (288.3, 62.7), turned to -90 degrees
- moved D43 158.3 mm to (288.5, 28.0)
- moved D30 153.1 mm to (29.1, 43.7), turned to 90 degrees
- moved D65 152.7 mm to (233.2, 78.7), turned to -90 degrees
- moved D46 150.7 mm to (43.3, 62.8), turned to -90 degrees
- moved D57 148.4 mm to (260.6, 62.6), turned to -90 degrees
- moved D42 147.9 mm to (262.2, 43.9), turned to 90 degrees
- moved D64 147.9 mm to (213.9, 78.7), turned to -90 degrees
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Connections:
- U1 pad 12: unconnected-(U1-PB7-Pad12) -> col8
- U1 pad 19: col8 -> unconnected-(U1-PD1-Pad19)
Routing:
- net row0: track 10.0 -> 578.4 mm, vias 0 -> 6
- net row1: track 11.3 -> 545.0 mm, vias 0 -> 4
- net row2: track 12.9 -> 480.1 mm, vias 0 -> 2
- net row4: track 0.00 -> 383.3 mm, vias 0 -> 5
- net row3: track 5.61 -> 357.7 mm, vias 1 -> 4
- net col0: track 5.99 -> 234.7 mm
- net col13: track 4.80 -> 230.2 mm, vias 0 -> 1
- net +5V: track 92.2 -> 304.6 mm
- net MOSI: track 4.66 -> 214.3 mm, vias 0 -> 2
- net col1: track 5.32 -> 214.0 mm
- net col12: track 6.08 -> 210.0 mm, vias 0 -> 2
- net GND: track 169.5 -> 353.4 mm, vias 7 -> 5
- net col11: track 5.99 -> 177.7 mm, vias 0 -> 1
- net MISO: track 4.00 -> 174.4 mm
- net SCK: track 3.34 -> 158.3 mm, vias 0 -> 2
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
Commit message: Small adjustement
Parts:
- moved SW44 0.28 mm to (289.5, 32.6)
Changed lines of the file:
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@@
 	(footprint "Button_Switch_Keyboard:SW_Cherry_MX_ISOEnter_PCB"
 		(layer "F.Cu")
-		(at 289.48175 32.3025)
+		(at 289.52 32.58)
 		(descr "Cherry MX keyswitch, ISO Enter, PCB mount, http://cherryamericas.com/wp-content/uploads/2014/12/mx_cat.pdf")
 		(tags "Cherry MX keyswitch ISO enter PCB")
@@
 	)
 	(segment
+		(start 16.87 5.09)
+		(end 17.38965 4.57035)
+		(width 0.3)
+		(layer "F.Cu")
+		(net 8)
+	)
+	(segment
+		(start 16.87 5.43)
+		(end 16.87 5.09)
+		(width 0.3)
+		(layer "F.Cu")
+		(net 8)
+	)
+	(segment
 		(start 22.254 4.57035)
-		(end 16.539 4.57035)
+		(end 17.38965 4.57035)
 		(width 0.3)
 		(layer "F.Cu")
@@
 	)
 	(via
-		(at 16.539 4.57035)
+		(at 22.254 4.57035)
 		(size 0.6)
 		(drill 0.3)
@@
 	)
 	(via
-		(at 22.254 4.57035)
+		(at 16.87 5.43)
 		(size 0.6)
 		(drill 0.3)
@@
 	)
 	(segment
-		(start 16.539 4.57035)
-		(end 16.539 5.139)
+		(start 16.87 5.47)
+		(end 17.936 6.536)
 		(width 0.3)
 		(layer "B.Cu")
@@
 	)
 	(segment
-		(start 17.936 6.536)
-		(end 17.936 9.8182)
+		(start 16.87 2.595)
+		(end 16.87 5.43)
 		(width 0.3)
 		(layer "B.Cu")
@@
 	)
 	(segment
-		(start 16.539 4.57035)
-		(end 16.87 4.23935)
+		(start 17.936 6.536)
+		(end 17.936 9.8182)
 		(width 0.3)
 		(layer "B.Cu")
@@
 	)
 	(segment
-		(start 16.539 5.139)
-		(end 17.936 6.536)
-		(width 0.3)
-		(layer "B.Cu")
-		(net 8)
-	)
-	(segment
 		(start 22.112175 4.57035)
 		(end 22.254 4.57035)
@@
 	)
 	(segment
-		(start 16.15825 9.7776)
-		(end 14.634 11.30185)
+		(start 16.87 5.43)
+		(end 16.87 5.47)
 		(width 0.3)
 		(layer "B.Cu")
@@
 	)
 	(segment
-		(start 14.634 11.30185)
-		(end 14.634 12.69835)
+		(start 16.15825 9.7776)
+		(end 14.634 11.30185)
 		(width 0.3)
 		(layer "B.Cu")
@@
 	)
 	(segment
-		(start 16.87 4.23935)
-		(end 16.87 2.595)
+		(start 14.634 11.30185)
+		(end 14.634 12.69835)
 		(width 0.3)
 		(layer "B.Cu")
@@
 	)
 	(segment
-		(start 290.1725 31.61175)
-		(end 289.48175 32.3025)
-		(width 0.2)
+		(start 290.1725 31.9275)
+		(end 289.52 32.58)
+		(width 0.3)
 		(layer "B.Cu")
 		(net 52)
@@
 	(segment
 		(start 290.1725 28.02)
-		(end 290.1725 31.61175)
-		(width 0.2)
+		(end 290.1725 31.9275)
+		(width 0.3)
 		(layer "B.Cu")
 		(net 52)

Commit message: Added gnd layers and ferrite bead on USB
Parts:
- added FB1: FerriteBead_Small, Inductor_SMD:L_0805_2012Metric_Pad1.15x1.40mm_HandSolder, B.Cu at (28.2, 1.31)
Connections:
- USB1 pad 13: GND -> Earth
Routing:
- net GND: track 353.4 -> 362.9 mm, vias 5 -> 30
- net col11: track 177.7 -> 178.6 mm
- net row0: track 578.4 -> 577.7 mm
- net col13: track 230.2 -> 230.7 mm
- net Earth: track 0.00 -> 0.32 mm, vias 0 -> 5
- added copper zone on B.Cu, net Earth
- added copper zone on F.Cu, net Earth
